File: kicad/bobbycar.kicad_pcb (KiCad board)
At the start: 2 copper layers, 42 x 45 mm, 48 parts, among them J1 Conn_01x04, J10 UART, J11 Conn_01x04, J12 CAN3, J13 CAN1, J15 CAN2, J2 PROG, J3 IO, J6 TFT, J7 I2C, J8 GAS, J9 BREMSE, U1 MPM3620, U3 ESP32-WROOM-32, U4 AMS1117-3.3, U7 MCP2542FDxMF

Commit message: Made files production ready
Parts:
- removed the R1 at (119.6, 70.5)
- removed the R16 at (131.3, 44.7)
- removed U7: MCP2542FDxMF, Package_DFN_QFN:DFN-8-1EP_3x3mm_P0.65mm_EP1.55x2.4mm
- added R12: 1k, Resistor_SMD:R_0603_1608Metric, F.Cu at (119.6, 70.5)
- added R15: 1k, Resistor_SMD:R_0603_1608Metric, F.Cu at (126.5, 53.2)
- added U2: TJA1051T-3, Package_SO:SOIC-8_3.9x4.9mm_P1.27mm, F.Cu at (132.6, 49.8)
- R10: renamed from R15; value 4k7 -> 2k2
- R11: value 1k -> 2k2
- R13: renamed from R2; value PULLDOWN -> 1k
- R16: renamed from R4; value PULLDOWN -> 1k
- R2: renamed from R13; value 1K -> 1k
- R3: renamed from R48; value 60R -> 56R
- R4: renamed from R49; value 60R -> 56R
- R9: renamed from R14; value 1K -> 1k
- moved R11 9.74 mm to (131.3, 44.7), turned to 0 degrees
- moved C4 4.00 mm to (134.5, 44.8)
- renumbered C43 to C1, C4 to C10, C10 to C11, C11 to C2, C12 to C3, C44 to C4, C45 to C5, C3 to C6, C2 to C7, C1 to C8, D12 to D1, D1 to D2, D2 to D3, J3 to J1, J13 to J10, J15 to J11, J2 to J12, J1 to J2, J8 to J3, J6 to J4, J11 to J5, J10 to J6, J9 to J7, J7 to J8, J12 to J9, R9 to R1, R10 to R14, R3 to R17, R12 to R18, U3 to U1, U1 to U3
Connections:
- R11 pad 1: IO0 -> SDA
Routing:
- net CAN_TX: track 16.5 -> 19.0 mm, vias 4 -> 2
- net CAN_RX: track 15.8 -> 14.7 mm
- net +5V: track 62.2 -> 63.1 mm
- net GND: vias 108 -> 107
Other:
- board text added: "3V3 GND"
- board text removed: "GND 3V3"

Commit message: grb
Parts:
- added Q1: SI2301CDS-T1-GE3, Package_TO_SOT_SMD:SOT-23, F.Cu at (124.5, 60.5)
- added R19: 2k2, Resistor_SMD:R_0603_1608Metric, F.Cu at (127.0, 60.5)
- R2, R9: value 1k -> 100r
Connections:
- J4 pad 8: TFT_LED -> Net-(J4-Pad8)
Routing:
- net TFT_LED: track 22.2 -> 30.0 mm, vias 1 -> 2
- net Net-(J4-Pad8): track 0.00 -> 3.62 mm
- net +3V3: track 116.5 -> 118.8 mm
- net GND: vias 107 -> 105
