File: kicad/bobbycar.sch (KiCad schematic (older format))
At the start: 47 parts, among them J1 Conn_01x04, J10 Conn_01x04, J11 Conn_01x04, J12 Conn_01x04, J13 Conn_01x04, J14 Conn_01x04, J15 Conn_01x04, J2 PROG, J3 Conn_01x13, J4 Conn_01x04, J5 19-39, J6 TFT, J7 Conn_01x04, J8 GAS, J9 BREMSE, U1 MPM3620, U3 ESP32-WROOM-32, U4 AMS1117-3.3, U7 MCP2542FDxMF

Commit message: created layout
Parts:
- removed J14, J4: Conn_01x04, Connector_PinHeader_2.54mm:PinHeader_1x04_P2.54mm_Vertical, symbol Connector_Generic:Conn_01x04
- removed J3: Conn_01x13, Connector_PinHeader_2.54mm:PinHeader_1x13_P2.54mm_Vertical, symbol Connector_Generic:Conn_01x13
- removed J5: 19-39, Connector_PinHeader_2.54mm:PinHeader_1x13_P2.54mm_Vertical, symbol Connector_Generic:Conn_01x13
- removed JP1, JP2: SolderJumper_2_Open, Jumper:SolderJumper-2_P1.3mm_Open_RoundedPad1.0x1.5mm, symbol Jumper:SolderJumper_2_Open
- added D1, D2: CDSOD323, Diode_SMD:D_SOD-323, symbol boardcomputer:CDSOD323
- added J3: IO, Connector_PinHeader_2.54mm:PinHeader_1x05_P2.54mm_Vertical, symbol Connector_Generic:Conn_01x05
- added R13, R14: 1K, Resistor_SMD:R_0603_1608Metric, symbol Device:R
- added R15, R16: 4k7, Resistor_SMD:R_0603_1608Metric, symbol Device:R
- J10: value Conn_01x04 -> UART; footprint (none) -> Connector_PinHeader_2.54mm:PinHeader_1x04_P2.54mm_Vertical
- J12: value Conn_01x04 -> CAN3; footprint (none) -> Connector_Molex:Molex_PicoBlade_53047-0410_1x04_P1.25mm_Vertical
- J13: value Conn_01x04 -> CAN1; footprint (none) -> Connector_PinHeader_2.54mm:PinHeader_1x04_P2.54mm_Vertical
- J15: value Conn_01x04 -> CAN2; footprint (none) -> Connector_PinHeader_2.54mm:PinHeader_1x04_P2.54mm_Vertical
- J7: value Conn_01x04 -> I2C; footprint (none) -> Connector_JST:JST_SH_SM04B-SRSS-TB_1x04-1MP_P1.00mm_Horizontal
Connections:
- wire segments 125 -> 120
Other:
- moved on the sheet: C1, C2, C44, C45, J1, J11, J12, J6, J7, J8

Commit message: Made files production ready
Parts:
- removed U7: MCP2542FDxMF, Package_DFN_QFN:DFN-8-1EP_3x3mm_P0.65mm_EP1.55x2.4mm, symbol Interface_CAN_LIN:MCP2542FDxMF
- added U2: TJA1051T-3, Package_SO:SOIC-8_3.9x4.9mm_P1.27mm, symbol Interface_CAN_LIN:TJA1051T-3
- C1: renamed from C43; LCSC Part # (none) -> C14663
- C10: renamed from C4; LCSC Part # (none) -> C45783
- C11: renamed from C10; LCSC Part # (none) -> C14663
- C2: renamed from C11; LCSC Part # (none) -> C19702
- C3: renamed from C12; LCSC Part # (none) -> C14663
- C4: renamed from C44; LCSC Part # (none) -> C14663
- C5: renamed from C45; LCSC Part # (none) -> C14663
- C6: renamed from C3; LCSC Part # (none) -> C15850
- C7: renamed from C2; LCSC Part # (none) -> C14663
- C8: renamed from C1; LCSC Part # (none) -> C14663
- C9: LCSC Part # (none) -> C14663
- D1: renamed from D12; LCSC Part # (none) -> C284104
- D2: renamed from D1; LCSC Part # (none) -> C127526
- D3: renamed from D2; LCSC Part # (none) -> C127526
- R1: renamed from R9; LCSC Part # (none) -> C21190
- R10: renamed from R15; value 4k7 -> 2k2; LCSC Part # (none) -> C4190
- R11: renamed from R16; value 4k7 -> 2k2; LCSC Part # (none) -> C4190
- R12: renamed from R1; value 100k -> 1k; LCSC Part # (none) -> C21190
- R13: renamed from R2; value PULLDOWN -> 1k; LCSC Part # (none) -> C21190
- R14: renamed from R10; LCSC Part # (none) -> C21190
- R15: renamed from R11; LCSC Part # (none) -> C21190
- R16: renamed from R4; value PULLDOWN -> 1k; LCSC Part # (none) -> C21190
- R17: renamed from R3; LCSC Part # (none) -> C22813
- R18: renamed from R12; LCSC Part # (none) -> C23000
- R2: renamed from R13; value 1K -> 1k; LCSC Part # (none) -> C21190
- R3: renamed from R48; value 60R -> 56R; LCSC Part # (none) -> C25196
- R4: renamed from R49; value 60R -> 56R; LCSC Part # (none) -> C25196
- R5, R6, R7, R8: LCSC Part # (none) -> C21190
- R9: renamed from R14; value 1K -> 1k; LCSC Part # (none) -> C21190
- U1: renamed from U3; LCSC Part # (none) -> C701343
- U4: LCSC Part # (none) -> C6186
- renumbered J3 to J1, J13 to J10, J15 to J11, J2 to J12, J1 to J2, J8 to J3, J6 to J4, J11 to J5, J10 to J6, J9 to J7, J7 to J8, J12 to J9, U1 to U3
Connections:
- net +3V3: now also U2.5 (VIO)
- net +5V: now also U2.3 (VCC)
- net CANH: now also U2.7 (CANH)
- net CANL: now also U2.6 (CANL)
- net CAN_RX: now also U2.4 (RXD)
- net CAN_TX: now also U2.1 (TXD)
- net GND: now also U2.2 (GND), U2.8 (S)
Other:
- moved on the sheet: C1, C4

Commit message: grb
Parts:
- added Q1: SI2301CDS-T1-GE3, Package_TO_SOT_SMD:SOT-23, symbol Transistor_FET:Si2319CDS
- added R19: 2k2, Resistor_SMD:R_0603_1608Metric, symbol Device:R
- C6: value 10uF -> 22uF; LCSC Part # C15850 -> C45783
- R2, R9: value 1k -> 100r; LCSC Part # C21190 -> C22775
Connections:
- net +3V3: now also Q1.2 (S), R19.2
- net TFT_LED: now also Q1.1 (G), R19.1; no longer J4.8 (Pin_8)
- new net: J4.8 (Pin_8), Q1.3 (D)
Other:
- moved on the sheet: J4
Changed lines of the file:
@@
 L Connector_Generic:Conn_01x09 J4
 U 1 1 5E855054
-P 4450 3250
-F 0 "J4" V 4667 3246 50  0000 C CNN
-F 1 "TFT" V 4576 3246 50  0000 C CNN
-F 2 "Connector_PinSocket_2.54mm:PinSocket_1x09_P2.54mm_Vertical" H 4450 3250 50  0001 C CNN
-F 3 "~" H 4450 3250 50  0001 C CNN
-	1    4450 3250
+P 4050 2400
+F 0 "J4" V 4267 2396 50  0000 C CNN
+F 1 "TFT" V 4176 2396 50  0000 C CNN
+F 2 "Connector_PinSocket_2.54mm:PinSocket_1x09_P2.54mm_Vertical" H 4050 2400 50  0001 C CNN
+F 3 "~" H 4050 2400 50  0001 C CNN
+	1    4050 2400
 	0    -1   -1   0
 $EndComp
@@
 L power:GND #PWR015
 U 1 1 5E857148
-P 4150 3450
-F 0 "#PWR015" H 4150 3200 50  0001 C CNN
-F 1 "GND" H 4150 3250 50  0000 C CNN
-F 2 "" H 4150 3450 50  0001 C CNN
-F 3 "" H 4150 3450 50  0001 C CNN
-	1    4150 3450
-	1    0    0    -1
-$EndComp
-Text GLabel 4250 3450 3    50   Input ~ 0
+P 3750 2600
+F 0 "#PWR015" H 3750 2350 50  0001 C CNN
+F 1 "GND" H 3750 2400 50  0000 C CNN
+F 2 "" H 3750 2600 50  0001 C CNN
+F 3 "" H 3750 2600 50  0001 C CNN
+	1    3750 2600
+	1    0    0    -1
+$EndComp
+Text GLabel 3850 2600 3    50   Input ~ 0
 CS
-Text GLabel 4350 3450 3    50   Input ~ 0
+Text GLabel 3950 2600 3    50   Input ~ 0
 TFT_RESET
-Text GLabel 4450 3450 3    50   Input ~ 0
+Text GLabel 4050 2600 3    50   Input ~ 0
 TFT_DC
-Text GLabel 4550 3450 3    50   Input ~ 0
+Text GLabel 4150 2600 3    50   Input ~ 0
 TFT_MOSI
-Text GLabel 4650 3450 3    50   Input ~ 0
+Text GLabel 4250 2600 3    50   Input ~ 0
 TFT_SCLK
-Text GLabel 4850 3450 3    50   Input ~ 0
+Text GLabel 4450 2600 3    50   Input ~ 0
 TFT_MISO
 Text GLabel 6350 4450 2    50   Input ~ 0
@@
 Text GLabel 2600 2900 2    50   Input ~ 0
 TFT_RESET
-Text GLabel 4750 3450 3    50   Input ~ 0
+Text GLabel 4050 3650 2    50   Input ~ 0
 TFT_LED
 Text GLabel 2600 4300 2    50   Input ~ 0
@@
 	9150 2550 9150 2650
 $Comp
-L Device:C C6
-U 1 1 601E68D1
-P 7150 2100
-F 0 "C6" H 7400 2150 50  0000 C CNN
-F 1 "10uF" H 7350 2050 50  0000 C CNN
-F 2 "Capacitor_SMD:C_0805_2012Metric" H 7188 1950 50  0001 C CNN
-F 3 "~" H 7150 2100 50  0001 C CNN
-F 4 "C15850	" H 7150 2100 50  0001 C CNN "LCSC Part #"
-	1    7150 2100
-	-1   0    0    1
-$EndComp
-$Comp
 L Device:C C10
 U 1 1 601E6C82
@@
 Connection ~ 7450 1950
 Wire Wire Line
-	7450 1950 7150 1950
-Wire Wire Line
 	7150 2250 7150 2350
 Wire Wire Line
@@
 Text GLabel 7000 1950 0    50   Input ~ 0
 15V
-Wire Wire Line
-	7000 1950 7150 1950
-Connection ~ 7150 1950
 $Comp
 L power:GND #PWR036
@@
 P 5600 5300
 F 0 "R9" H 5670 5346 50  0000 L CNN
-F 1 "1k" V 5500 5250 50  0000 L CNN
+F 1 "100r" V 5500 5250 50  0000 L CNN
 F 2 "Resistor_SMD:R_0603_1608Metric" V 5530 5300 50  0001 C CNN
 F 3 "~" H 5600 5300 50  0001 C CNN
-F 4 "C21190" H 5600 5300 50  0001 C CNN "LCSC Part #"
+F 4 "C22775" H 5600 5300 50  0001 C CNN "LCSC Part #"
 	1    5600 5300
 	0    1    1    0
@@
 L power:+5V #PWR014
 U 1 1 5E857D53
-P 4050 3450
-F 0 "#PWR014" H 4050 3300 50  0001 C CNN
-F 1 "+5V" H 4150 3650 50  0000 C CNN
-F 2 "" H 4050 3450 50  0001 C CNN
-F 3 "" H 4050 3450 50  0001 C CNN
-	1    4050 3450
+P 3650 2600
+F 0 "#PWR014" H 3650 2450 50  0001 C CNN
+F 1 "+5V" H 3750 2800 50  0000 C CNN
+F 2 "" H 3650 2600 50  0001 C CNN
+F 3 "" H 3650 2600 50  0001 C CNN
+	1    3650 2600
 	-1   0    0    1
 $EndComp
@@
 P 4300 5300
 F 0 "R2" H 4370 5346 50  0000 L CNN
-F 1 "1k" V 4200 5250 50  0000 L CNN
+F 1 "100r" V 4200 5250 50  0000 L CNN
 F 2 "Resistor_SMD:R_0603_1608Metric" V 4230 5300 50  0001 C CNN
 F 3 "~" H 4300 5300 50  0001 C CNN
-F 4 "C21190" H 4300 5300 50  0001 C CNN "LCSC Part #"
+F 4 "C22775" H 4300 5300 50  0001 C CNN "LCSC Part #"
 	1    4300 5300
 	0    1    1    0
 $EndComp
+$Comp
+L Transistor_FET:Si2319CDS Q1
+U 1 1 603F8418
+P 4050 3450
+F 0 "Q1" V 4392 3450 50  0000 C CNN
+F 1 "SI2301CDS-T1-GE3" V 4301 3450 50  0000 C CNN
+F 2 "Package_TO_SOT_SMD:SOT-23" H 4250 3375 50  0001 L CIN
+F 3 "https://datasheet.lcsc.com/szlcsc/Vishay-Intertech-SI2301CDS-T1-GE3_C10487.pdf" H 4050 3450 50  0001 L CNN
+F 4 "C10487" H 4050 3450 50  0001 C CNN "LCSC Part #"
+	1    4050 3450
+	0    1    -1   0
+$EndComp
+$Comp
+L power:+3V3 #PWR039
+U 1 1 604120E1
+P 3550 3350
+F 0 "#PWR039" H 3550 3200 50  0001 C CNN
+F 1 "+3V3" H 3565 3523 50  0000 C CNN
+F 2 "" H 3550 3350 50  0001 C CNN
+F 3 "" H 3550 3350 50  0001 C CNN
+	1    3550 3350
+	1    0    0    -1
+$EndComp
+Wire Wire Line
+	4350 2600 4350 3350
+Wire Wire Line
+	4350 3350 4250 3350
+Wire Wire Line
+	4050 3650 3750 3650
+Wire Wire Line
+	3550 3350 3750 3350
+$Comp
+L Device:R R19
+U 1 1 6041F00A
+P 3750 3500
+F 0 "R19" V 4000 3450 50  0000 L CNN
+F 1 "2k2" V 4000 3250 50  0000 L CNN
+F 2 "Resistor_SMD:R_0603_1608Metric" V 3680 3500 50  0001 C CNN
+F 3 "~" H 3750 3500 50  0001 C CNN
+F 4 "C4190" H 3750 3500 50  0001 C CNN "LCSC Part #"
+	1    3750 3500
+	-1   0    0    1
+$EndComp
+Connection ~ 3750 3350
+Wire Wire Line
+	3750 3350 3850 3350
+Wire Wire Line
+	7000 1950 7150 1950
+$Comp
+L Device:C C6
+U 1 1 6043AF8C
+P 7150 2100
+F 0 "C6" H 7050 2200 50  0000 C CNN
+F 1 "22uF" H 7050 2000 50  0000 C CNN
+F 2 "Capacitor_SMD:C_0805_2012Metric" H 7188 1950 50  0001 C CNN
+F 3 "~" H 7150 2100 50  0001 C CNN
+F 4 "C45783" H 7150 2100 50  0001 C CNN "LCSC Part #"
+	1    7150 2100
+	-1   0    0    1
+$EndComp
+Connection ~ 7150 1950
+Wire Wire Line
+	7150 1950 7450 1950
 $EndSCHEMATC
