File: kicad/bobbycar.sch (KiCad schematic (older format))
At the start: 54 parts, among them J1 IO, J11 CAN2, J12 PROG, J2 IO2, J3 GAS, J4 TFT, J5 Conn_01x04, J7 BREMSE, J8 I2C, J9 CAN3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

Commit message: changed to single 3.3V dcdc
Parts:
- removed C1: 100n, Capacitor_SMD:C_0603_1608Metric, symbol Device:C
- removed C10, C6: 22uF, Capacitor_SMD:C_0805_2012Metric, symbol Device:C
- removed C12: 10n, Capacitor_SMD:C_0603_1608Metric, symbol Device:C
- removed D4: B230A, Diode_SMD:D_SMA, symbol Diode:B230
- removed J5: Conn_01x04, Connector_PinHeader_2.54mm:PinHeader_1x04_P2.54mm_Vertical, symbol Connector_Generic:Conn_01x04
- removed L1: 4.7uH, boardcomputer:L_5040, symbol Device:L_Small
- removed R12: 1k, Resistor_SMD:R_0603_1608Metric, symbol Device:R
- removed R17: 49.9k, Resistor_SMD:R_0603_1608Metric, symbol Device:R
- removed R18: 9.53k, Resistor_SMD:R_0603_1608Metric, symbol Device:R
- removed U2: TJA1051T-3, Package_SO:SOIC-8_3.9x4.9mm_P1.27mm, symbol Interface_CAN_LIN:TJA1051T-3
- removed U3: MPM2359, Package_TO_SOT_SMD:SOT-23-6, symbol boardcomputer:MPM2359
- added U2: SN65HVD231, Package_SO:SOIC-8_3.9x4.9mm_P1.27mm, symbol Interface_CAN_LIN:SN65HVD231
- D2: LCSC Part # C127526 -> C139300
- J1: footprint Connector_PinHeader_2.54mm:PinHeader_1x05_P2.54mm_Vertical -> Connector_PinHeader_2.54mm:PinHeader_1x07_P2.54mm_Vertical; symbol Connector_Generic:Conn_01x05 -> Connector_Generic:Conn_01x07
- J2: footprint Connector_PinHeader_2.54mm:PinHeader_1x04_P2.54mm_Vertical -> Connector_PinHeader_2.54mm:PinHeader_1x06_P2.54mm_Vertical; symbol Connector_Generic:Conn_01x04 -> Connector_Generic:Conn_01x06
Connections:
- net +3V3: now also C4.1, J1.1 (Pin_1), J2.1 (Pin_1), J4.1 (Pin_1), U2.3 (VCC)
- net 15V: now also C13.2, R5.2, U5.5 (IN)
- net CANH: now also U2.7 (CANH)
- net CANL: now also U2.6 (CANL)
- net CAN_RX: now also U2.4 (R)
- net CAN_TX: now also U2.1 (D)
- net GND: now also J1.7 (Pin_7), J2.6 (Pin_6), U2.2 (GND), U2.8 (Rs)
- net IO18: now also J1.4 (Pin_4); no longer J1.2 (Pin_2)
- net IO19: now also J1.3 (Pin_3); no longer J1.1 (Pin_1)
- net IO25: now also J2.4 (Pin_4); no longer J2.3 (Pin_3)
- net IO26: now also J2.5 (Pin_5); no longer J2.4 (Pin_4)
- net IO27: now also J1.2 (Pin_2); no longer J1.5 (Pin_5)
- net IO32: now also J2.2 (Pin_2); no longer J2.1 (Pin_1)
- net IO33: now also J2.3 (Pin_3); no longer J2.2 (Pin_2)
- net IO4: now also J1.6 (Pin_6); no longer J1.4 (Pin_4)
- net IO5: now also J1.5 (Pin_5); no longer J1.3 (Pin_3)
- removed net +5V: C13.2, C4.1, J4.1 (Pin_1), R5.2, U5.5 (IN)
