File: kicad/bobbycar.kicad_sch (KiCad schematic)
At the start: 51 parts, among them J1 IO, J11 CAN2, J12 PROG, J2 IO2, J3 GAS, J4 TFT, J7 BREMSE, J8 I2C, J9 CAN3, Q1 SI2301CDS-T1-GE3, U1 ESP32-WROOM-32, U2 SN65HVD231, U5 MPM2359

Commit message: added 16 buttons
Parts:
- removed D2, D3: CDSOD323, Diode_SMD:D_SOD-323, symbol boardcomputer:CDSOD323
- removed J8: I2C, Connector_JST:JST_SH_SM04B-SRSS-TB_1x04-1MP_P1.00mm_Horizontal, symbol Connector_Generic:Conn_01x04
- added BZ1: Buzzer, Capacitor_SMD:CP_Elec_18x22, symbol Device:Buzzer
- added C1, C6: 100n, Capacitor_SMD:C_0603_1608Metric, symbol Device:C
- added D14: D, symbol Device:D
- added J10: BREMSE, Connector_PinHeader_2.54mm:PinHeader_1x03_P2.54mm_Vertical, symbol Connector_Generic:Conn_01x03
- added J13: LED, Connector_JST:JST_XH_B3B-XH-A_1x03_P2.50mm_Vertical, symbol Connector_Generic:Conn_01x03
- added J5, J6: Conn_02x08_Odd_Even, Connector_PinHeader_2.54mm:PinHeader_2x08_P2.54mm_Vertical, symbol Connector_Generic:Conn_02x08_Odd_Even
- added J8: GAS, Connector_PinHeader_2.54mm:PinHeader_1x03_P2.54mm_Vertical, symbol Connector_Generic:Conn_01x03
- added Q2, Q3: SI2301CDS-T1-GE3, Package_TO_SOT_SMD:SOT-23, symbol Transistor_FET:Si2319CDS
- added R12: 100r, Resistor_SMD:R_0603_1608Metric, symbol Device:R
- added R17: 1k, Resistor_SMD:R_0603_1608Metric, symbol Device:R
- added R8: 100k, Resistor_SMD:R_0603_1608Metric, symbol Device:R
- added U3, U4, U6, U7, U8: USBLC6-4SC6, Package_TO_SOT_SMD:SOT-23-6, symbol Power_Protection:USBLC6-4SC6
- J12: footprint Connector_PinHeader_2.54mm:PinHeader_1x05_P2.54mm_Vertical -> Connector_JST:JST_XH_B6B-XH-A_1x06_P2.50mm_Vertical; symbol Connector_Generic:Conn_01x05 -> Connector_Generic:Conn_01x06
- J2: symbol Connector_Generic:Conn_01x06 -> Connector_Generic:Conn_01x07
- R10: value 2k2 -> 100k; LCSC Part # C4190 -> C21190
- R11: value 2k2 -> 100r; LCSC Part # C4190 -> C22775
- R13, R16: value 1k -> 100k
- gave numbers to parts that had none: 8
Connections:
- net IO18 is gone; now on net IN2: J1.4 (Pin_4), U1.30 (IO18)
- net IO27 is gone; now on net IN3: J1.2 (Pin_2), U1.12 (IO27)
- net IO4 is gone; now on net IN1: J1.6 (Pin_6), U1.26 (IO4)
- net OUT1 is gone; now on net IO19: D10.3 (K), D12.3 (K), D4.3 (K), D8.3 (K)
- net OUT2 is gone; now on net IO5: D11.3 (K), D13.3 (K), D7.3 (K), D9.3 (K)
- net +3V3: now also J10.1 (Pin_1), J8.1 (Pin_1), R17.2, U3.5 (VBUS), U4.5 (VBUS), U6.5 (VBUS), U7.5 (VBUS), U8.5 (VBUS); no longer R10.2, R11.2
- net 15V: now also D14.1 (K), J13.3 (Pin_3)
- net B1: now also J5.1 (Pin_1), U3.1 (I/O1)
- net B10: now also D10.2 (A), J6.4 (Pin_4), U6.3 (I/O2); no longer D11.1 (K)
- net B11: now also D11.1 (K), J6.6 (Pin_6), U6.4 (I/O3); no longer D11.2 (A)
- net B12: now also D11.2 (A), J6.8 (Pin_8), U6.6 (I/O4); no longer D10.2 (A)
- net B13: now also J6.10 (Pin_10), U7.1 (I/O1)
- net B14: now also D12.2 (A), J6.12 (Pin_12), U7.3 (I/O2); no longer D13.1 (K)
- net B15: now also D13.1 (K), J6.14 (Pin_14), U7.4 (I/O3); no longer D13.2 (A)
- net B16: now also D13.2 (A), J6.16 (Pin_16), U7.6 (I/O4); no longer D12.2 (A)
- net B2: now also D4.2 (A), J5.3 (Pin_3), U3.3 (I/O2); no longer D7.1 (K)
- net B3: now also D7.1 (K), J5.5 (Pin_5), U3.4 (I/O3); no longer D4.2 (A)
- net B4: now also J5.7 (Pin_7), U3.6 (I/O4)
- net B5: now also J5.9 (Pin_9), U4.1 (I/O1)
- net B6: now also D8.2 (A), J5.11 (Pin_11), U4.3 (I/O2); no longer D9.1 (K)
- net B7: now also D9.1 (K), J5.13 (Pin_13), U4.4 (I/O3); no longer D8.2 (A)
- net B8: now also J5.15 (Pin_15), U4.6 (I/O4)
- net B9: now also J6.2 (Pin_2), U6.1 (I/O1)
- net GND: now also J2.7 (Pin_7), R10.2, BZ1.2 (+), C1.1, C6.1, J10.3 (Pin_3), J13.1 (Pin_1), J8.3 (Pin_3), Q2.3 (D), Q3.3 (D), R8.2, U3.2 (GND), U4.2 (GND), U6.2 (GND), U7.2 (GND), U8.2 (GND); no longer J2.6 (Pin_6)
- net IN1: now also J5.2 (Pin_2), J5.4 (Pin_4), J5.6 (Pin_6), J5.8 (Pin_8)
- net IN2: now also J5.10 (Pin_10), J5.12 (Pin_12), J5.14 (Pin_14), J5.16 (Pin_16)
- net IN3: now also J6.1 (Pin_1), J6.3 (Pin_3), J6.5 (Pin_5), J6.7 (Pin_7)
- net IN4: now also U1.27 (IO16), J6.11 (Pin_11), J6.13 (Pin_13), J6.15 (Pin_15), J6.9 (Pin_9)
- net IO0: now also Q2.1 (G)
- net IO33: now also J13.2 (Pin_2)
- net RAW_BREMSE: now also U8.3 (I/O2)
- net RAW_GAS: now also U8.1 (I/O1)
- net IO36 renamed RAW_M365_GAS
- net RAW_M365_GAS: now also R11.1, C1.2, R8.1, U8.4 (I/O3)
- net IO39 renamed RAW_M365_BREMS
- net RAW_M365_BREMS: now also R10.1, C6.2, R12.1, U8.6 (I/O4)
- net SCL renamed IO17
- net IO17: now also J2.6 (Pin_6); no longer R10.1
- removed net SDA: R11.1, U1.27 (IO16)
- new net: D14.2 (A), J12.6 (Pin_6)
- new net: Q2.2 (S), Q3.1 (G), R17.1
- new net: J8.2 (Pin_2), R11.2
- new net: J10.2 (Pin_2), R12.2
- new net BUZZER: BZ1.1 (-), Q3.2 (S)
Other:
- note added: "0V - 15V"
- note added: "Button"
- note added: "Buttons"
- note added: "GPIO"
- note added: "LED / GPIO"
- note added: "Save to plug in with 5V"
- note added: "excluded"
- moved on the sheet: C7, C8, J1, J3, J7, J9, R13, R16, R2, R9

Commit message: Add H-bridge for beeper; convert symbol library to new format
Parts:
- removed Q2, Q3: SI2301CDS-T1-GE3, Package_TO_SOT_SMD:SOT-23, symbol Transistor_FET:Si2319CDS
- removed R17: 1k, Resistor_SMD:R_0603_1608Metric, symbol Device:R
- added C? (x2): (no value), symbol Device:C
- added Q? (x2): Q_Dual_NMOS_S1G1D2S2G2D1, symbol Device:Q_Dual_NMOS_S1G1D2S2G2D1
- added R? (x4): (no value), symbol Device:R
- added U?: DGD05473FN-7, symbol boardcomputer:DGD05473FN-7
- BZ1: value Buzzer -> (none); footprint Capacitor_SMD:CP_Elec_18x22 -> (none)
- C1, C3, C4, C5, C6, C7, C8: value 100n -> (none); footprint Capacitor_SMD:C_0603_1608Metric -> (none)
- C13, C15: value 22uF -> (none); footprint Capacitor_SMD:C_0805_2012Metric -> (none)
- C14: value 10n -> (none); footprint Capacitor_SMD:C_0603_1608Metric -> (none)
- C2: value 10u -> (none); footprint Capacitor_SMD:C_0603_1608Metric -> (none)
- D1: value NUP2105L -> (none); footprint Package_TO_SOT_SMD:SOT-23 -> (none)
- D10, D11, D12, D13, D4, D7, D8, D9: value BAV99 -> (none); footprint Package_TO_SOT_SMD:SOT-23 -> (none)
- D14: value D -> (none)
- D5, D6: value B230A -> (none); footprint Diode_SMD:D_SMA -> (none)
- J1: value IO -> (none); footprint Connector_PinHeader_2.54mm:PinHeader_1x07_P2.54mm_Vertical -> (none)
- J10, J7: value BREMSE -> (none); footprint Connector_PinHeader_2.54mm:PinHeader_1x03_P2.54mm_Vertical -> (none)
- J11: value CAN2 -> (none); footprint Connector_JST:JST_XH_B4B-XH-A_1x04_P2.50mm_Vertical -> (none)
- J12: value PROG -> (none); footprint Connector_JST:JST_XH_B6B-XH-A_1x06_P2.50mm_Vertical -> (none)
- J13: value LED -> (none); footprint Connector_JST:JST_XH_B3B-XH-A_1x03_P2.50mm_Vertical -> (none)
- J2: value IO2 -> (none); footprint Connector_PinHeader_2.54mm:PinHeader_1x06_P2.54mm_Vertical -> (none)
- J3, J8: value GAS -> (none); footprint Connector_PinHeader_2.54mm:PinHeader_1x03_P2.54mm_Vertical -> (none)
- J4: value TFT -> (none); footprint Connector_PinSocket_2.54mm:PinSocket_1x09_P2.54mm_Vertical -> (none)
- J5, J6: value Conn_02x08_Odd_Even -> (none); footprint Connector_PinHeader_2.54mm:PinHeader_2x08_P2.54mm_Vertical -> (none)
- J9: value CAN3 -> (none); footprint Connector_Molex:Molex_PicoBlade_53047-0410_1x04_P1.25mm_Vertical -> (none)
- L2: value 4.7uH -> (none); footprint boardcomputer:L_5040 -> (none)
- Q1: value SI2301CDS-T1-GE3 -> (none); footprint Package_TO_SOT_SMD:SOT-23 -> (none)
- R1, R14, R15, R5: value 1k -> (none); footprint Resistor_SMD:R_0603_1608Metric -> (none)
- R10, R13, R16, R8: value 100k -> (none); footprint Resistor_SMD:R_0603_1608Metric -> (none)
- R11, R12, R2, R9: value 100r -> (none); footprint Resistor_SMD:R_0603_1608Metric -> (none)
- R19: value 2k2 -> (none); footprint Resistor_SMD:R_0603_1608Metric -> (none)
- R3, R4: value 56R -> (none); footprint Resistor_SMD:R_0603_1608Metric -> (none)
- R6: value 49.9k -> (none); footprint Resistor_SMD:R_0603_1608Metric -> (none)
- R7: value 16.2k -> (none); footprint Resistor_SMD:R_0603_1608Metric -> (none)
- U1: value ESP32-WROOM-32 -> (none); footprint RF_Module:ESP32-WROOM-32 -> (none)
- U2: value SN65HVD231 -> (none); footprint Package_SO:SOIC-8_3.9x4.9mm_P1.27mm -> (none)
- U3, U4, U6, U7, U8: value USBLC6-4SC6 -> (none); footprint Package_TO_SOT_SMD:SOT-23-6 -> (none)
- U5: value MPM2359 -> (none); footprint Package_TO_SOT_SMD:SOT-23-6 -> (none)
Connections:
- net +3V3: now also Q?.6 (D), U?.1 (VCC), U?.7 (EN)
- net BUZZER: now also C?.2, R?.1
- net GND: now also Q?.4 (S), R?.2, R?.2, U?.11 (COM), U?.9 (COM)
- net IO0: now also U?.8 (IN)
- new net: C?.1, C?.1, Q?.1 (S), Q?.3 (D), U?.4 (VS)
- new net: C?.2, U?.2 (VB)
- new net: R?.1, U?.6 (DT)
- new net: R?.1, U?.3 (HO)
- new net: Q?.2 (G), R?.2
- new net: R?.1, U?.10 (LO)
- new net: Q?.5 (G), R?.2
Other:
- moved on the sheet: BZ1

Commit message: Correct part number for MOSFET driver
Parts:
- BZ1: value (none) -> Buzzer; footprint (none) -> Capacitor_SMD:CP_Elec_18x22
- C1, C3, C4, C5, C6, C7, C8: value (none) -> 100n; footprint (none) -> Capacitor_SMD:C_0603_1608Metric
- C13, C15, C?: value (none) -> 22uF; footprint (none) -> Capacitor_SMD:C_0805_2012Metric
- C14: value (none) -> 10n; footprint (none) -> Capacitor_SMD:C_0603_1608Metric
- C2: value (none) -> 10u; footprint (none) -> Capacitor_SMD:C_0603_1608Metric
- C?: value (none) -> 1u
- D1: value (none) -> NUP2105L; footprint (none) -> Package_TO_SOT_SMD:SOT-23
- D10, D11, D12, D13, D4, D7, D8, D9: value (none) -> BAV99; footprint (none) -> Package_TO_SOT_SMD:SOT-23
- D14: value (none) -> D
- D5, D6: value (none) -> B230A; footprint (none) -> Diode_SMD:D_SMA
- J1: value (none) -> IO; footprint (none) -> Connector_PinHeader_2.54mm:PinHeader_1x07_P2.54mm_Vertical
- J10, J7: value (none) -> BREMSE; footprint (none) -> Connector_PinHeader_2.54mm:PinHeader_1x03_P2.54mm_Vertical
- J11: value (none) -> CAN2; footprint (none) -> Connector_JST:JST_XH_B4B-XH-A_1x04_P2.50mm_Vertical
- J12: value (none) -> PROG; footprint (none) -> Connector_JST:JST_XH_B6B-XH-A_1x06_P2.50mm_Vertical
- J13: value (none) -> LED; footprint (none) -> Connector_JST:JST_XH_B3B-XH-A_1x03_P2.50mm_Vertical
- J2: value (none) -> IO2; footprint (none) -> Connector_PinHeader_2.54mm:PinHeader_1x06_P2.54mm_Vertical
- J3, J8: value (none) -> GAS; footprint (none) -> Connector_PinHeader_2.54mm:PinHeader_1x03_P2.54mm_Vertical
- J4: value (none) -> TFT; footprint (none) -> Connector_PinSocket_2.54mm:PinSocket_1x09_P2.54mm_Vertical
- J5, J6: value (none) -> Conn_02x08_Odd_Even; footprint (none) -> Connector_PinHeader_2.54mm:PinHeader_2x08_P2.54mm_Vertical
- J9: value (none) -> CAN3; footprint (none) -> Connector_Molex:Molex_PicoBlade_53047-0410_1x04_P1.25mm_Vertical
- L2: value (none) -> 4.7uH; footprint (none) -> boardcomputer:L_5040
- Q1: value (none) -> SI2301CDS-T1-GE3; footprint (none) -> Package_TO_SOT_SMD:SOT-23
- Q?: footprint (none) -> Package_TO_SOT_SMD:SOT-363_SC-70-6
- R1, R14, R15, R5: value (none) -> 1k; footprint (none) -> Resistor_SMD:R_0603_1608Metric
- R10, R13, R16, R8, R?: value (none) -> 100k; footprint (none) -> Resistor_SMD:R_0603_1608Metric
- R11, R12, R2, R9: value (none) -> 100r; footprint (none) -> Resistor_SMD:R_0603_1608Metric
- R19: value (none) -> 2k2; footprint (none) -> Resistor_SMD:R_0603_1608Metric
- R3, R4, R? (x2): value (none) -> 56R; footprint (none) -> Resistor_SMD:R_0603_1608Metric
- R6: value (none) -> 49.9k; footprint (none) -> Resistor_SMD:R_0603_1608Metric
- R7: value (none) -> 16.2k; footprint (none) -> Resistor_SMD:R_0603_1608Metric
- R?: value (none) -> 4.7k
- U: renamed from U?; value DGD05473FN-7 -> (none); symbol boardcomputer:DGD05473FN-7 -> boardcomputer:DGD0506AFN-7
- U1: value (none) -> ESP32-WROOM-32; footprint (none) -> RF_Module:ESP32-WROOM-32
- U2: value (none) -> SN65HVD231; footprint (none) -> Package_SO:SOIC-8_3.9x4.9mm_P1.27mm
- U3, U4, U6, U7, U8: value (none) -> USBLC6-4SC6; footprint (none) -> Package_TO_SOT_SMD:SOT-23-6
- U5: value (none) -> MPM2359; footprint (none) -> Package_TO_SOT_SMD:SOT-23-6
