File: kicad/bobbycar.kicad_sch (KiCad schematic)
At the start: 66 parts, among them J10 BREMSE, J11 CAN2, J12 PROG, J13 LED, J2 IO2, J3 GAS, J4 TFT, J5 Conn_02x08_Odd_Even, J6 Conn_02x08_Odd_Even, J7 BREMSE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

Commit message: Cleared pcb, added usb c
Parts:
- added C9: 100n, Capacitor_SMD:C_0603_1608Metric, symbol Device:C
- added D2: D, Diode_SMD:D_SOD-123, symbol Device:D
- added JP2, JP3, JP4, JP5: SolderJumper_2_Open, Jumper:SolderJumper-2_P1.3mm_Open_RoundedPad1.0x1.5mm, symbol Jumper:SolderJumper_2_Open
- added Q2, Q3: SS8050_C2150, Package_TO_SOT_SMD:TSOT-23, symbol SS8050:SS8050_C2150
- added R17, R18: 5k1, Resistor_SMD:R_0603_1608Metric, symbol Device:R
- added R20, R22: 12k, Resistor_SMD:R_0603_1608Metric, symbol Device:R
- added U10: CH343G, Package_SO:SOIC-16_3.9x9.9mm_P1.27mm, symbol wch-usb-uart:CH343G
- added USBC1: MC-311D, USB-C-SMD_MC-311D, symbol usb_c_bobby:MC-311D
- J2: footprint Connector_PinHeader_2.54mm:PinHeader_1x06_P2.54mm_Vertical -> Connector_PinHeader_2.54mm:PinHeader_1x07_P2.54mm_Vertical
- R1, R15: value 1k -> 10k; LCSC (none) -> C25804; LCSC Part # C21190 -> (none)
Connections:
- net +3V3: now also R1.2, JP2.1 (A), U10.15 (VIO); no longer Q1.2 (S), R1.1
- net 15V: now also D2.1 (K)
- net EN: now also R1.1, Q2.3 (C); no longer R1.2
- net ESP_RX: now also U10.2 (TXD)
- net ESP_TX: now also U10.3 (RXD)
- net GND: now also C9.1, JP5.1 (A), R17.2, R18.1, U10.1 (GND), USBC1.1 (SHIELD), USBC1.2 (SHIELD), USBC1.3 (SHIELD), USBC1.4 (SHIELD), USBC1.A1-B12 (GND), USBC1.B1-A12 (GND)
- net IO0: now also Q3.2 (E)
- net TFT_LED: no longer Q1.1 (G), R19.1
- net at J4.8 (Pin_8): now also JP3.1 (A), JP4.1 (A); no longer Q1.3 (D)
- new net: Q1.1 (G), R19.1
- new net: JP2.2 (B), JP3.2 (B), Q1.2 (S)
- new net: JP4.2 (B), JP5.2 (B), Q1.3 (D)
- new net: R17.1, USBC1.A5 (CC1)
- new net: R18.2, USBC1.B5 (CC2)
- new net: Q3.1 (B), R22.2
- new net: C9.2, U10.4 (V3)
- new net: Q2.1 (B), R20.2
- new net +5V: D2.2 (A), U10.16 (VDD5), U10.7 (VBUS), USBC1.A4-B9 (VBUS), USBC1.B4-A9 (VBUS)
- new net DTR: Q3.3 (C), R20.1, U10.10 (~{DTR}/TNOW)
- new net RTS: Q2.2 (E), R22.1, U10.11 (~{RTS})
- new net USB_DN: U10.6 (UD-), USBC1.A7 (DN1), USBC1.B7 (DN2)
- new net USB_DP: U10.5 (UD+), USBC1.A6 (DP1), USBC1.B6 (DP2)
- no-connect marks 0 -> 5
Other:
- note added: "RED DISPLAY: Bridge JP2 & JP4 BLACK DISPLAY: Bridge JP3 & JP5"
- moved on the sheet: J2, Q1, R19

Commit message: Layout done
Parts:
- removed BZ1: Buzzer, Capacitor_SMD:CP_Elec_18x22, symbol Device:Buzzer
- removed C10: 1u, Capacitor_SMD:C_0805_2012Metric, symbol Device:C
- removed D14: D, Diode_SMD:D_SOD-123, symbol Device:D
- removed J12: PROG, Connector_JST:JST_XH_B6B-XH-A_1x06_P2.50mm_Vertical, symbol Connector_Generic:Conn_01x06
- removed JP1: Jumper_2_Open, Jumper:SolderJumper-2_P1.3mm_Open_RoundedPad1.0x1.5mm, symbol Jumper:Jumper_2_Open
- removed R21: 4.7k, Resistor_SMD:R_0603_1608Metric, symbol Device:R
- removed U9: MCP1416, Package_TO_SOT_SMD:SOT-23-5, symbol Driver_FET:MCP1416
- J2: footprint Connector_PinHeader_2.54mm:PinHeader_1x07_P2.54mm_Vertical -> boardcomputer:PinHeader_2x04_P2.54mm_Vertical_7Pin
Connections:
- net +3V3: now also J10.3 (Pin_3), J3.3 (Pin_3), J7.3 (Pin_3), J8.3 (Pin_3); no longer J10.1 (Pin_1), J3.1 (Pin_1), J7.1 (Pin_1), J8.1 (Pin_1)
- net GND: now also J10.1 (Pin_1), J3.1 (Pin_1), J7.1 (Pin_1), J8.1 (Pin_1); no longer J10.3 (Pin_3), J3.3 (Pin_3), J7.3 (Pin_3), J8.3 (Pin_3)
Other:
- note removed: "0V - 15V"
- note removed: "Save to plug in with 5V"

Commit message: Half done trace layout
Connections:
- net TFT_LED: now also Q1.1 (G), R19.1
Changed lines of the file:
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@@
     )
   )
-  (global_label "TFT_LED" (shape input) (at 111.76 100.33 0) (fields_autoplaced)
+  (global_label "TFT_LED" (shape input) (at 101.6 107.95 0) (fields_autoplaced)
     (effects (font (size 1.27 1.27)) (justify left))
-    (property "Referenzen zwischen Schaltplänen" "${INTERSHEET_REFS}" (id 0) (at 8.89 7.62 0)
+    (property "Referenzen zwischen Schaltplänen" "${INTERSHEET_REFS}" (id 0) (at -1.27 15.24 0)
       (effects (font (size 1.27 1.27)) hide)
     )
